File: mike_pcb_motors/mike_pcb_motors.sch (KiCad schematic (older format))
At the start: 13 parts, among them J1 Motor1, J2 Motor2, J3 Motor3, J4 Motor1, J5 Screw_Terminal_01x02, J6 Motor2, J7 PCB_connector, U1 MDD3A-3ADCMD, U2 MDD3A-3ADCMD, U3 SBX-DRIVER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

Commit message: Updating the design files
Parts:
- J4: value Motor1 -> CraneMotorGear1
- J6: value Motor2 -> CraneMotorHook1
Other:
- moved on the sheet: A2, J1, J2, J3, J4, J5, J6, J7, U1, U2, U3, U5

Commit message: Updating PCB files, baseplate file
Parts:
- added C1, C2: C, Capacitor_THT:C_Radial_D8.0mm_H7.0mm_P3.50mm, symbol Device:C
- added J8, J9: Conn_01x03_Male, Connector_PinHeader_2.54mm:PinHeader_1x03_P2.54mm_Vertical, symbol Connector:Conn_01x03_Male
Connections:
- net +5V: now also C2.2, J8.2 (Pin_2), J9.2 (Pin_2)
- net GND: now also C1.1, C2.1, J8.3 (Pin_3), J9.3 (Pin_3)
- net VCC: now also C1.2
- net Servo_PWM1: now reaches A2.6 (D3)
- net Servo_PWM1: now also J8.1 (Pin_1)
- net Servo_PWM2: now reaches A2.8 (D5)
- net Servo_PWM2: now also J9.1 (Pin_1)
Changed lines of the file:
@@
 	1    0    0    -1
 $EndComp
+$Comp
+L power:VCC #PWR0133
+U 1 1 61D47EFB
+P 9950 4400
+F 0 "#PWR0133" H 9950 4250 50  0001 C CNN
+F 1 "VCC" V 9965 4527 50  0000 L CNN
+F 2 "" H 9950 4400 50  0001 C CNN
+F 3 "" H 9950 4400 50  0001 C CNN
+	1    9950 4400
+	0    -1   -1   0
+$EndComp
+$Comp
+L power:GND #PWR0134
+U 1 1 61D4856F
+P 10350 4450
+F 0 "#PWR0134" H 10350 4200 50  0001 C CNN
+F 1 "GND" V 10355 4322 50  0000 R CNN
+F 2 "" H 10350 4450 50  0001 C CNN
+F 3 "" H 10350 4450 50  0001 C CNN
+	1    10350 4450
+	1    0    0    -1
+$EndComp
+Wire Wire Line
+	10250 4400 10350 4400
+Wire Wire Line
+	10350 4400 10350 4450
+$Comp
+L Device:C C2
+U 1 1 61D4B8A1
+P 10400 3800
+F 0 "C2" V 10148 3800 50  0000 C CNN
+F 1 "C" V 10239 3800 50  0000 C CNN
+F 2 "Capacitor_THT:C_Radial_D8.0mm_H7.0mm_P3.50mm" H 10438 3650 50  0001 C CNN
+F 3 "~" H 10400 3800 50  0001 C CNN
+	1    10400 3800
+	0    1    1    0
+$EndComp
+$Comp
+L power:GND #PWR0135
+U 1 1 61D4B8AD
+P 10650 3850
+F 0 "#PWR0135" H 10650 3600 50  0001 C CNN
+F 1 "GND" V 10655 3722 50  0000 R CNN
+F 2 "" H 10650 3850 50  0001 C CNN
+F 3 "" H 10650 3850 50  0001 C CNN
+	1    10650 3850
+	1    0    0    -1
+$EndComp
+Wire Wire Line
+	10550 3800 10650 3800
+Wire Wire Line
+	10650 3800 10650 3850
+$Comp
+L power:+5V #PWR0136
+U 1 1 61D4C0D9
+P 10150 3800
+F 0 "#PWR0136" H 10150 3650 50  0001 C CNN
+F 1 "+5V" H 10165 3973 50  0000 C CNN
+F 2 "" H 10150 3800 50  0001 C CNN
+F 3 "" H 10150 3800 50  0001 C CNN
+	1    10150 3800
+	0    -1   -1   0
+$EndComp
+Wire Wire Line
+	10150 3800 10250 3800
+$Comp
+L Device:C C1
+U 1 1 61D4E08B
+P 10100 4400
+F 0 "C1" V 9848 4400 50  0000 C CNN
+F 1 "C" V 9939 4400 50  0000 C CNN
+F 2 "Capacitor_THT:C_Radial_D8.0mm_H7.0mm_P3.50mm" H 10138 4250 50  0001 C CNN
+F 3 "~" H 10100 4400 50  0001 C CNN
+	1    10100 4400
+	0    1    1    0
+$EndComp
+$Comp
+L Connector:Conn_01x03_Male J8
+U 1 1 61D4F0F3
+P 1550 6400
+F 0 "J8" H 1658 6681 50  0000 C CNN
+F 1 "Conn_01x03_Male" H 1658 6590 50  0000 C CNN
+F 2 "Connector_PinHeader_2.54mm:PinHeader_1x03_P2.54mm_Vertical" H 1550 6400 50  0001 C CNN
+F 3 "~" H 1550 6400 50  0001 C CNN
+	1    1550 6400
+	1    0    0    -1
+$EndComp
+$Comp
+L Connector:Conn_01x03_Male J9
+U 1 1 61D51007
+P 3500 6400
+F 0 "J9" H 3608 6681 50  0000 C CNN
+F 1 "Conn_01x03_Male" H 3608 6590 50  0000 C CNN
+F 2 "Connector_PinHeader_2.54mm:PinHeader_1x03_P2.54mm_Vertical" H 3500 6400 50  0001 C CNN
+F 3 "~" H 3500 6400 50  0001 C CNN
+	1    3500 6400
+	1    0    0    -1
+$EndComp
+$Comp
+L power:+5V #PWR0137
+U 1 1 61D52241
+P 3800 6400
+F 0 "#PWR0137" H 3800 6250 50  0001 C CNN
+F 1 "+5V" H 3815 6573 50  0000 C CNN
+F 2 "" H 3800 6400 50  0001 C CNN
+F 3 "" H 3800 6400 50  0001 C CNN
+	1    3800 6400
+	0    1    1    0
+$EndComp
+$Comp
+L power:GND #PWR0138
+U 1 1 61D532EE
+P 3800 6500
+F 0 "#PWR0138" H 3800 6250 50  0001 C CNN
+F 1 "GND" V 3805 6372 50  0000 R CNN
+F 2 "" H 3800 6500 50  0001 C CNN
+F 3 "" H 3800 6500 50  0001 C CNN
+	1    3800 6500
+	1    0    0    -1
+$EndComp
+Text GLabel 4100 1950 0    50   Input ~ 0
+Servo_PWM1
+Text GLabel 4100 2150 0    50   Input ~ 0
+Servo_PWM2
+Text GLabel 4050 6300 2    50   Input ~ 0
+Servo_PWM2
+Wire Wire Line
+	4050 6300 3700 6300
+Wire Wire Line
+	3800 6400 3700 6400
+Wire Wire Line
+	3800 6500 3700 6500
+$Comp
+L power:+5V #PWR0139
+U 1 1 61D56A50
+P 1850 6400
+F 0 "#PWR0139" H 1850 6250 50  0001 C CNN
+F 1 "+5V" H 1865 6573 50  0000 C CNN
+F 2 "" H 1850 6400 50  0001 C CNN
+F 3 "" H 1850 6400 50  0001 C CNN
+	1    1850 6400
+	0    1    1    0
+$EndComp
+$Comp
+L power:GND #PWR0140
+U 1 1 61D56A56
+P 1850 6500
+F 0 "#PWR0140" H 1850 6250 50  0001 C CNN
+F 1 "GND" V 1855 6372 50  0000 R CNN
+F 2 "" H 1850 6500 50  0001 C CNN
+F 3 "" H 1850 6500 50  0001 C CNN
+	1    1850 6500
+	1    0    0    -1
+$EndComp
+Text GLabel 2100 6300 2    50   Input ~ 0
+Servo_PWM1
+Wire Wire Line
+	2100 6300 1750 6300
+Wire Wire Line
+	1850 6400 1750 6400
+Wire Wire Line
+	1850 6500 1750 6500
 $EndSCHEMATC

Commit message: CAD changes
Changes to top and bottom platform
Parts:
- J1, J2, J3, J4, J6, J7: symbol Connector:Conn_01x06_Male -> Connector:Conn_01x06_Female
- J8, J9: symbol Connector:Conn_01x03_Male -> Connector:Conn_01x03_Female
Changed lines of the file:
@@
 SDA_5V
 $Comp
-L Connector:Conn_01x06_Male J1
+L Connector:Conn_01x06_Female J1
 U 1 1 60EE8352
 P 6500 1750
@@
 F 3 "~" H 6500 1750 50  0001 C CNN
 	1    6500 1750
-	1    0    0    -1
+	-1   0    0    -1
 $EndComp
 $Comp
@@
 Motor1_B
 $Comp
-L Connector:Conn_01x06_Male J2
+L Connector:Conn_01x06_Female J2
 U 1 1 60EED123
 P 6500 2650
@@
 F 3 "~" H 6500 2650 50  0001 C CNN
 	1    6500 2650
-	1    0    0    -1
+	-1   0    0    -1
 $EndComp
 $Comp
@@
 Motor2_B
 $Comp
-L Connector:Conn_01x06_Male J3
+L Connector:Conn_01x06_Female J3
 U 1 1 60EEDD8F
 P 6500 3550
@@
 F 3 "~" H 6500 3550 50  0001 C CNN
 	1    6500 3550
-	1    0    0    -1
+	-1   0    0    -1
 $EndComp
 $Comp
@@
 CraneMotor2_PWM2
 $Comp
-L Connector:Conn_01x06_Male J4
+L Connector:Conn_01x06_Female J4
 U 1 1 61C28ED1
 P 1200 4200
@@
 F 3 "~" H 1200 4200 50  0001 C CNN
 	1    1200 4200
-	1    0    0    -1
+	-1   0    0    -1
 $EndComp
 $Comp
@@
 CraneMotor1_B
 $Comp
-L Connector:Conn_01x06_Male J6
+L Connector:Conn_01x06_Female J6
 U 1 1 61C28EE7
 P 1250 5150
@@
 F 3 "~" H 1250 5150 50  0001 C CNN
 	1    1250 5150
-	1    0    0    -1
+	-1   0    0    -1
 $EndComp
 $Comp
@@
 CraneMotor2_B
 $Comp
-L Connector:Conn_01x06_Male J7
+L Connector:Conn_01x06_Female J7
 U 1 1 61C4BD88
 P 8200 5100
@@
 F 3 "~" H 8200 5100 50  0001 C CNN
 	1    8200 5100
-	1    0    0    -1
+	-1   0    0    -1
 $EndComp
 $Comp
@@
 $EndComp
 $Comp
-L Connector:Conn_01x03_Male J8
+L Connector:Conn_01x03_Female J8
 U 1 1 61D4F0F3
 P 1550 6400
@@
 F 3 "~" H 1550 6400 50  0001 C CNN
 	1    1550 6400
-	1    0    0    -1
-$EndComp
-$Comp
-L Connector:Conn_01x03_Male J9
+	-1   0    0    -1
+$EndComp
+$Comp
+L Connector:Conn_01x03_Female J9
 U 1 1 61D51007
 P 3500 6400
@@
 F 3 "~" H 3500 6400 50  0001 C CNN
 	1    3500 6400
-	1    0    0    -1
-$EndComp
-$Comp
+	-1   0    0    -1
+$EndComp
+$Comp
