File: mike_pcb_motors/mike_pcb_motors.kicad_pcb (KiCad board)
At the start: 2 copper layers, 125 x 91.1 mm, 13 parts, among them J1 Motor1, J2 Motor2, J3 Motor3, J4 Motor1, J5 Screw_Terminal_01x02, J6 Motor2, J7 PCB_connector, U1 MDD3A-3ADCMD, U2 MDD3A-3ADCMD, U3 SBX-DRIVER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

Commit message: Updating the design files
Parts:
- moved J3 2.77 mm to (117.8, 123.2)
- moved J7 1.59 mm to (183.1, 123.0)
Routing:
- net +5V: track 0.00 -> 331.1 mm, vias 0 -> 8
- net VCC: track 0.00 -> 197.1 mm, vias 0 -> 2
- net SCL_5V: track 0.00 -> 154.7 mm, vias 0 -> 3
- net SDA_5V: track 0.00 -> 131.8 mm, vias 0 -> 5
- net CraneMotor1_M2: track 0.00 -> 116.5 mm
- net CraneMotor1_M1: track 0.00 -> 95.4 mm, vias 0 -> 2
- net Motor2_PWM1: track 0.00 -> 92.4 mm, vias 0 -> 4
- net Motor3_PWM1: track 0.00 -> 88.3 mm
- net Motor2_PWM2: track 0.00 -> 87.2 mm, vias 0 -> 4
- net Motor1_PWM2: track 0.00 -> 84.7 mm, vias 0 -> 4
- net CraneMotor2_M2: track 0.00 -> 82.8 mm, vias 0 -> 2
- net Motor1_PWM1: track 0.00 -> 76.2 mm, vias 0 -> 4
- net Motor3_PWM2: track 0.00 -> 72.7 mm
- net Motor3_B: track 0.00 -> 69.4 mm, vias 0 -> 4
- net CraneMotor1_B: track 0.00 -> 66.4 mm, vias 0 -> 2
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
Commit message: Updating PCB files, baseplate file
Parts:
- added C1: C, Capacitor_THT:C_Radial_D8.0mm_H7.0mm_P3.50mm, F.Cu at (165.1, 191.1)
- added C2: C, Capacitor_THT:C_Radial_D8.0mm_H7.0mm_P3.50mm, F.Cu at (189.6, 211.5)
- added J8: Conn_01x03_Male, Connector_PinHeader_2.54mm:PinHeader_1x03_P2.54mm_Vertical, F.Cu at (128.4, 218.6)
- added J9: Conn_01x03_Male, Connector_PinHeader_2.54mm:PinHeader_1x03_P2.54mm_Vertical, F.Cu at (128.4, 215.8)
- added REF**: MountingHole_3.2mm_M3_DIN965, MountingHole:MountingHole_3.2mm_M3_DIN965, F.Cu at (92.8, 157.3)
- added REF**: MountingHole_3.2mm_M3_DIN965, MountingHole:MountingHole_3.2mm_M3_DIN965, F.Cu at (186.1, 175.1)
- added REF**: MountingHole_3.2mm_M3_DIN965, MountingHole:MountingHole_3.2mm_M3_DIN965, F.Cu at (186.9, 144.2)
- added REF**: MountingHole_3.2mm_M3_DIN965, MountingHole:MountingHole_3.2mm_M3_DIN965, F.Cu at (79.0, 144.3)
- J4: value Motor1 -> CraneMotorGear1
- J6: value Motor2 -> CraneMotorHook1
- moved J2 13.2 mm to (139.6, 136.7)
- moved A1 13.2 mm to (122.0, 148.0)
- moved A2 13.2 mm to (93.5, 206.7)
- moved J1 13.2 mm to (159.0, 136.7)
- moved J3 13.2 mm to (116.2, 136.3)
- moved J4 13.2 mm to (84.0, 187.2)
- moved J5 13.2 mm to (185.5, 188.7)
- moved J6 13.2 mm to (84.0, 189.7)
- moved J7 13.2 mm to (181.6, 136.2)
- moved U1 13.2 mm to (112.5, 161.7)
- moved U2 13.2 mm to (147.2, 162.2)
- moved U3 13.2 mm to (148.3, 196.7)
- moved U5 13.2 mm to (172.4, 206.4)
Connections:
- A2 pad 6: Net-(A2-Pad6) -> Servo_PWM1
- A2 pad 8: Net-(A2-Pad8) -> Servo_PWM2
Routing:
- net +5V: track 331.1 -> 395.7 mm, vias 8 -> 10
- net GND: track 35.7 -> 99.0 mm, vias 9 -> 22
- net Servo_PWM1: track 0.00 -> 28.0 mm
- net Servo_PWM2: track 0.00 -> 22.2 mm
- net Motor3_PWM1: track 88.3 -> 76.5 mm
- net VCC: track 197.1 -> 205.4 mm, vias 2 -> 4
- net CraneMotor2_PWM1: track 36.6 -> 38.9 mm
- net CraneMotor2_PWM2: track 31.8 -> 34.0 mm
- net Motor1_B: track 62.1 -> 63.4 mm
- net CraneMotor1_PWM1: track 40.4 -> 39.3 mm
- net CraneMotor1_PWM2: track 40.1 -> 40.6 mm
- added copper zone on B.Cu, net Net-(U1-Pad4)
- added copper zone on B.Cu, net Net-(U2-Pad6)

Commit message: Updating the production files
Routing:
- net GND: track 99.0 -> 107.1 mm, vias 22 -> 24
Changed lines of the file:
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@@
     (thickness 1.6)
     (drawings 99)
-    (tracks 543)
+    (tracks 550)
     (zones 0)
     (modules 21)
@@
     (mod_text_size 1 1)
     (mod_text_width 0.15)
-    (pad_size 2.7 1.7)
+    (pad_size 2 2)
     (pad_drill 1)
     (pad_to_mask_clearance 0)
@@
     (visible_elements 7FFFFFFF)
     (pcbplotparams
-      (layerselection 0x010fc_ffffffff)
+      (layerselection 0x01000_ffffffff)
       (usegerberextensions false)
       (usegerberattributes true)
@@
       (drillshape 0)
       (scaleselection 1)
-      (outputdirectory "LMR-Gerbrer/"))
+      (outputdirectory "mike_pcb_motors-Gerbrer/"))
   )
   (net 0 "")
@@
       (effects (font (size 1 1) (thickness 0.15)))
     )
-    (pad 2 thru_hole circle (at 3.5 0 180) (size 2 2) (drill 0.8) (layers *.Cu *.Mask)
+    (pad 2 thru_hole circle (at 3.5 0 180) (size 2 2) (drill 1) (layers *.Cu *.Mask)
       (net 3 +5V))
-    (pad 1 thru_hole circle (at 0 0 180) (size 2 2) (drill 0.8) (layers *.Cu *.Mask)
+    (pad 1 thru_hole circle (at 0 0 180) (size 2 2) (drill 1) (layers *.Cu *.Mask)
       (net 5 GND))
     (model ${KISYS3DMOD}/Capacitor_THT.3dshapes/C_Radial_D8.0mm_H7.0mm_P3.50mm.wrl
@@
       (effects (font (size 1 1) (thickness 0.15)))
     )
-    (pad 2 thru_hole circle (at 3.5 0) (size 2 2) (drill 0.8) (layers *.Cu *.Mask)
+    (pad 2 thru_hole circle (at 3.5 0) (size 2 2) (drill 1) (layers *.Cu *.Mask)
       (net 54 VCC))
-    (pad 1 thru_hole circle (at 0 0) (size 2 2) (drill 0.8) (layers *.Cu *.Mask)
+    (pad 1 thru_hole circle (at 0 0) (size 2 2) (drill 1) (layers *.Cu *.Mask)
       (net 5 GND))
     (model ${KISYS3DMOD}/Capacitor_THT.3dshapes/C_Radial_D8.0mm_H7.0mm_P3.50mm.wrl
@@
   (segment (start 180.375 206.305) (end 171.02 215.66) (width 2) (layer B.Cu) (net 3))
   (segment (start 189.15 197.53) (end 180.375 206.305) (width 2) (layer B.Cu) (net 3))
-  (via (at 131.73 213.23) (size 2.1) (drill 1) (layers F.Cu B.Cu) (net 3))
-  (segment (start 131.73 213.23) (end 140.3 204.66) (width 2) (layer F.Cu) (net 3))
   (via (at 166.16 212.35) (size 2.1) (drill 1) (layers F.Cu B.Cu) (net 3))
-  (segment (start 158.47 204.66) (end 166.16 212.35) (width 2) (layer F.Cu) (net 3))
-  (segment (start 140.3 204.66) (end 158.47 204.66) (width 2) (layer F.Cu) (net 3))
   (segment (start 166.16 215.49) (end 166.33 215.66) (width 2) (layer B.Cu) (net 3))
-  (segment (start 166.16 212.35) (end 166.16 215.49) (width 2) (layer B.Cu) (net 3))
   (segment (start 130.96 215.87) (end 130.98 215.85) (width 2) (layer B.Cu) (net 3))
   (segment (start 130.96 218.63) (end 130.96 215.87) (width 2) (layer B.Cu) (net 3))
-  (segment (start 130.98 213.98) (end 131.73 213.23) (width 2) (layer B.Cu) (net 3))
-  (segment (start 130.98 215.85) (end 130.98 213.98) (width 2) (layer B.Cu) (net 3))
   (segment (start 105.25 133.07) (end 106.08 133.9) (width 1) (layer B.Cu) (net 3))
   (segment (start 76.19 133.07) (end 105.25 133.07) (width 1) (layer B.Cu) (net 3))
@@
   (segment (start 87.53 171.33) (end 70.08 171.33) (width 1) (layer B.Cu) (net 3))
   (segment (start 93.47 177.27) (end 87.53 171.33) (width 1) (layer B.Cu) (net 3))
+  (segment (start 158.47 204.66) (end 166.16 212.35) (width 2) (layer F.Cu) (net 3))
+  (segment (start 140.3 204.66) (end 158.47 204.66) (width 2) (layer F.Cu) (net 3))
+  (segment (start 166.16 212.35) (end 166.16 215.49) (width 2) (layer B.Cu) (net 3))
+  (via (at 131.73 213.23) (size 2.1) (drill 1) (layers F.Cu B.Cu) (net 3))
+  (segment (start 130.98 215.85) (end 130.98 213.98) (width 2) (layer B.Cu) (net 3))
+  (segment (start 130.98 213.98) (end 131.73 213.23) (width 2) (layer B.Cu) (net 3))
+  (segment (start 131.73 213.23) (end 140.3 204.66) (width 2) (layer F.Cu) (net 3))
   (via (at 176.39 171.21) (size 2.1) (drill 1) (layers F.Cu B.Cu) (net 4))
   (segment (start 181.035 166.565) (end 176.39 171.21) (width 0.5) (layer B.Cu) (net 4))
@@
   (segment (start 136.64 215.85) (end 136.75 215.74) (width 2) (layer B.Cu) (net 5))
   (segment (start 133.52 215.85) (end 136.64 215.85) (width 2) (layer B.Cu) (net 5))
+  (segment (start 178.99 215.66) (end 179.04 215.71) (width 2) (layer B.Cu) (net 5))
+  (segment (start 176.49 215.66) (end 178.99 215.66) (width 2) (layer B.Cu) (net 5))
+  (via (at 180.91 213.7) (size 2.1) (drill 1) (layers F.Cu B.Cu) (net 5))
+  (segment (start 179.04 215.57) (end 180.91 213.7) (width 2) (layer B.Cu) (net 5))
+  (segment (start 179.04 215.71) (end 179.04 215.57) (width 2) (layer B.Cu) (net 5))
+  (via (at 180.91 210.88) (size 2.1) (drill 1) (layers F.Cu B.Cu) (net 5))
+  (segment (start 180.91 213.7) (end 180.91 210.88) (width 2) (layer B.Cu) (net 5))
   (via (at 178.49 173.11) (size 2.1) (drill 1) (layers F.Cu B.Cu) (net 6))
   (segment (start 182.495 169.105) (end 178.49 173.11) (width 0.5) (layer B.Cu) (net 6))
@@
   (via (at 144.93 210.159998) (size 2.1) (drill 1) (layers F.Cu B.Cu) (net 67))
   (segment (start 149.930002 215.16) (end 144.93 210.159998) (width 0.5) (layer F.Cu) (net 67))
+  (segment (start 125.92 209.59) (end 144.360002 209.59) (width 0.5) (layer B.Cu) (net 67))
+  (segment (start 123.97 206.66) (end 123.97 207.64) (width 0.5) (layer B.Cu) (net 67))
+  (segment (start 123.97 207.64) (end 125.92 209.59) (width 0.5) (layer B.Cu) (net 67))
   (segment (start 144.360002 209.59) (end 144.93 210.159998) (width 0.5) (layer B.Cu) (net 67))
-  (segment (start 125.92 209.59) (end 144.360002 209.59) (width 0.5) (layer B.Cu) (net 67))
-  (segment (start 123.97 207.64) (end 125.92 209.59) (width 0.5) (layer B.Cu) (net 67))
-  (segment (start 123.97 206.66) (end 123.97 207.64) (width 0.5) (layer B.Cu) (net 67))
-  (segment (start 121.43 207.42) (end 121.43 206.66) (width 0.5) (layer B.Cu) (net 68))
   (segment (start 124.57 210.56) (end 121.43 207.42) (width 0.5) (layer B.Cu) (net 68))
   (segment (start 142.1 210.56) (end 124.57 210.56) (width 0.5) (layer B.Cu) (net 68))
   (segment (start 144.48 212.94) (end 142.1 210.56) (width 0.5) (layer B.Cu) (net 68))
   (segment (start 144.48 220.795) (end 144.48 212.94) (width 0.5) (layer B.Cu) (net 68))
+  (segment (start 121.43 207.42) (end 121.43 206.66) (width 0.5) (layer B.Cu) (net 68))
   (via (at 79.72 179.74) (size 2.1) (drill 1) (layers F.Cu B.Cu) (net 69))
   (via (at 78.2 184.23) (size 2.1) (drill 1) (layers F.Cu B.Cu) (net 69))
@@
   (segment (start 114.61 202.38) (end 92.98 202.38) (width 0.5) (layer B.Cu) (net 69))
   (segment (start 118.89 206.66) (end 114.61 202.38) (width 0.5) (layer B.Cu) (net 69))
+  (segment (start 117.7 211.6) (end 140.13 211.6) (width 0.5) (layer B.Cu) (net 70))
   (segment (start 141.94 213.41) (end 141.94 220.795) (width 0.5) (layer B.Cu) (net 70))
+  (segment (start 113.81 206.66) (end 113.81 207.71) (width 0.5) (layer B.Cu) (net 70))
+  (segment (start 113.81 207.71) (end 117.7 211.6) (width 0.5) (layer B.Cu) (net 70))
   (segment (start 140.13 211.6) (end 141.94 213.41) (width 0.5) (layer B.Cu) (net 70))
-  (segment (start 117.7 211.6) (end 140.13 211.6) (width 0.5) (layer B.Cu) (net 70))
-  (segment (start 113.81 207.71) (end 117.7 211.6) (width 0.5) (layer B.Cu) (net 70))
-  (segment (start 113.81 206.66) (end 113.81 207.71) (width 0.5) (layer B.Cu) (net 70))
   (via (at 108.58 204.25) (size 2.1) (drill 1) (layers F.Cu B.Cu) (net 71))
   (segment (start 108.73 206.66) (end 108.73 204.4) (width 0.5) (layer B.Cu) (net 71))
@@
   (segment (start 139.95 197.07) (end 139.95 196.66) (width 1.5) (layer B.Cu) (net 79))
   (segment (start 138.54 198.48) (end 139.95 197.07) (width 1.5) (layer B.Cu) (net 79))
+  (segment (start 111.27 208.05) (end 111.27 206.66) (width 0.5) (layer B.Cu) (net 80))
+  (segment (start 115.84 212.62) (end 111.27 208.05) (width 0.5) (layer B.Cu) (net 80))
+  (segment (start 125.92 212.62) (end 115.84 212.62) (width 0.5) (layer B.Cu) (net 80))
+  (segment (start 128.44 215.14) (end 125.92 212.62) (width 0.5) (layer B.Cu) (net 80))
   (segment (start 128.44 215.85) (end 128.44 215.14) (width 0.5) (layer B.Cu) (net 80))
-  (segment (start 128.44 215.14) (end 126.14 212.84) (width 0.5) (layer B.Cu) (net 80))
-  (segment (start 126.14 212.84) (end 116.06 212.84) (width 0.5) (layer B.Cu) (net 80))
-  (segment (start 111.27 208.05) (end 111.27 206.66) (width 0.5) (layer B.Cu) (net 80))
-  (segment (start 116.06 212.84) (end 111.27 208.05) (width 0.5) (layer B.Cu) (net 80))
   (segment (start 106.19 208.01) (end 106.19 206.66) (width 0.5) (layer B.Cu) (net 81))
-  (segment (start 112.29 214.11) (end 106.19 208.01) (width 0.5) (layer B.Cu) (net 81))
-  (segment (start 122.16 214.11) (end 112.29 214.11) (width 0.5) (layer B.Cu) (net 81))
-  (segment (start 126.68 218.63) (end 122.16 214.11) (width 0.5) (layer B.Cu) (net 81))
+  (segment (start 111.97 213.79) (end 106.19 208.01) (width 0.5) (layer B.Cu) (net 81))
+  (segment (start 121.84 213.79) (end 111.97 213.79) (width 0.5) (layer B.Cu) (net 81))
+  (segment (start 126.68 218.63) (end 121.84 213.79) (width 0.5) (layer B.Cu) (net 81))
   (segment (start 128.42 218.63) (end 126.68 218.63) (width 0.5) (layer B.Cu) (net 81))
   (zone (net 5) (net_name GND) (layer F.Cu) (hatch edge 0.508)
