File: mike_pcb_arduino_sheild/mike_pcb_arduino_sheild.kicad_pcb (KiCad board)
At the start: 2 copper layers, 49.9 x 53.6 mm, 2 parts, among them J101 Conn_01x06_Male

Commit message: Updating the code and pcb files
Routing:
- added copper zone on F.Cu, net GND
- removed copper zone on F.Cu, net (none)
