File: mike_pcb_control/mike_pcb_control.kicad_pcb (KiCad board)
At the start: 2 copper layers, 102.2 x 72.7 mm, 5 parts, among them J1 Conn_01x06_Male, J4 Raspberry_Pi_2_3, U3 LLC-4channel, U4 Adafruit_Feather_Pinout

Commit message: Updating the design files
Parts:
- added C1: C, Capacitor_THT:C_Radial_D8.0mm_H7.0mm_P3.50mm, F.Cu at (90.3, 65.7)
- added J2: Conn_01x06_Male, Connector_PinHeader_2.54mm:PinHeader_1x06_P2.54mm_Vertical, F.Cu at (88.5, 45.5)
- added J3: Conn_01x03_Male, Connector_PinHeader_2.54mm:PinHeader_1x03_P2.54mm_Vertical, F.Cu at (98.7, 53.3)
- added J5: Conn_01x03_Male, Connector_PinHeader_2.54mm:PinHeader_1x03_P2.54mm_Vertical, F.Cu at (94.0, 53.3)
- moved J1 71.3 mm to (107.1, 61.2), turned to 270 degrees
- moved U4 52.7 mm to (141.7, 90.8)
- moved A2 50.2 mm to (93.8, 89.1)
- moved U3 0.71 mm to (114.0, 52.5)
Connections:
- A2 pad 19: Net-(A2-Pad19) -> A0
- A2 pad 20: Net-(A2-Pad20) -> A1
- A2 pad 23: SDA_IMU -> SDA5V
- A2 pad 24: SCL_IMU -> SCL5V
- U4 pad 17: SDA_IMU -> SDA3V3
- U4 pad 18: SCL_IMU -> SCL3V3
Routing:
- net +5V: track 0.00 -> 203.9 mm, vias 0 -> 2
- net SDA3V3: track 0.00 -> 109.3 mm
- net SCL3V3: track 0.00 -> 102.8 mm, vias 0 -> 2
- net TX3V3: track 0.00 -> 70.6 mm
- net RX3V3: track 0.00 -> 59.9 mm
- net GND: track 0.00 -> 58.0 mm, vias 0 -> 11
- net +3V3: track 0.00 -> 47.6 mm
- net A0: track 0.00 -> 40.2 mm, vias 0 -> 2
- net A1: track 0.00 -> 34.8 mm, vias 0 -> 2
- net SCL5V: track 0.00 -> 33.4 mm, vias 0 -> 2
- net +3.3VA: track 0.00 -> 30.0 mm
- net TX5V: track 0.00 -> 26.3 mm
- net SDA5V: track 0.00 -> 25.7 mm
- net RX5V: track 0.00 -> 17.2 mm

Commit message: Updating PCB files, baseplate file
Parts:
- added REF**: MountingHole_3.2mm_M3, MountingHole:MountingHole_3.2mm_M3, F.Cu at (131.0, 48.7)
- added REF**: MountingHole_3.2mm_M3, MountingHole:MountingHole_3.2mm_M3, F.Cu at (165.3, 50.3)
- added REF**: MountingHole_3.2mm_M3, MountingHole:MountingHole_3.2mm_M3, F.Cu at (137.8, 29.6)
- moved C1 31.6 mm to (90.0, 34.0)
- moved A2 31.6 mm to (93.6, 57.4)
- moved J1 31.6 mm to (106.9, 29.6)
- moved J2 31.6 mm to (88.3, 13.9)
- moved J3 31.6 mm to (98.5, 21.6)
- moved J4 31.6 mm to (150.8, 3.86)
- moved J5 31.6 mm to (93.8, 21.6)
- moved U3 31.6 mm to (113.8, 20.9)
- moved U4 31.6 mm to (141.5, 59.2)
Routing:
- net +5V: track 203.9 -> 200.8 mm
- net GND: track 58.0 -> 61.0 mm, vias 11 -> 12
- net RX3V3: track 59.9 -> 59.0 mm
- net +3.3VA: track 30.0 -> 29.4 mm
- added copper zone on B.Cu, net Net-(U4-Pad9)

Commit message: PCB bugfix, I2C seperated
I2C for IMU seperated from main I2C bus
Parts:
- removed REF** (x3): MountingHole_3.2mm_M3, MountingHole:MountingHole_3.2mm_M3
Connections:
- A2 pad 1: Net-(A2-Pad1) -> TX-RX_link
- A2 pad 2: Net-(A2-Pad2) -> RX5V
- A2 pad 23: SDA5V -> SDA_IMU
- A2 pad 24: SCL5V -> SCL_IMU
- J2 pad 1: RX5V -> TX-RX_link
- U3 pad 11: SCL5V -> SDA5V
- U3 pad 12: SDA5V -> SCL5V
- U4 pad 17: SDA3V3 -> SDA_IMU
- U4 pad 18: SCL3V3 -> SCL_IMU
Routing:
- net SCL_IMU: track 0.00 -> 91.7 mm
- net SDA_IMU: track 0.00 -> 78.7 mm
- net TX-RX_link: track 0.00 -> 49.1 mm, vias 0 -> 1
- net RX5V: track 17.2 -> 63.2 mm, vias 0 -> 2
- net SCL3V3: track 102.8 -> 64.9 mm, vias 2 -> 0
- net SDA3V3: track 109.3 -> 78.7 mm
- net GND: track 61.0 -> 85.9 mm, vias 12 -> 9
- net SCL5V: track 33.4 -> 9.99 mm, vias 2 -> 0
- net +5V: track 200.8 -> 187.2 mm, vias 2 -> 0
- net SDA5V: track 25.7 -> 24.5 mm
- net A1: track 34.8 -> 33.8 mm
- net A0: track 40.1 -> 39.3 mm
- added copper zone on B.Cu, net (none)
- removed copper zone on B.Cu, net Net-(U4-Pad9)

Commit message: Updating the PCB files
Routing:
- added copper zone on B.Cu, net Net-(U4-Pad8)
- removed copper zone on B.Cu, net (none)
